Commit message: Correctly implemented Panda Arm
Tested on moveit

File: src/robot_arm/panda_description/urdf/control/panda_hand.ros2_control.xacro (robot description, xacro)
@@ -4,14 +4,7 @@
         <ros2_control name="${name}" type="system">
             <hardware>
-                <xacro:if value="${ros2_control_hardware_type == 'mock_components'}">
-                    <plugin>mock_components/GenericSystem</plugin>
-                </xacro:if>
-                <xacro:if value="${ros2_control_hardware_type == 'isaac'}">
-                    <plugin>topic_based_ros2_control/TopicBasedSystem</plugin>
-                    <param name="joint_commands_topic">/isaac_joint_commands</param>
-                    <param name="joint_states_topic">/isaac_joint_states</param>
-                </xacro:if>
+                <plugin>gz_ros2_control/GazeboSimSystem</plugin>
             </hardware>
-            <joint name="panda_finger_joint1">
+              <joint name="panda_finger_joint1">
                 <command_interface name="position" />
                 <state_interface name="position">

File: src/robot_arm/panda_description/urdf/panda.ros2_control.xacro (robot description, xacro)
@@ -5,12 +5,5 @@
         <ros2_control name="${name}" type="system">
             <hardware>
-                <xacro:if value="${ros2_control_hardware_type == 'mock_components'}">
-                    <plugin>mock_components/GenericSystem</plugin>
-                </xacro:if>
-                <xacro:if value="${ros2_control_hardware_type == 'isaac'}">
-                    <plugin>topic_based_ros2_control/TopicBasedSystem</plugin>
-                    <param name="joint_commands_topic">/isaac_joint_commands</param>
-                    <param name="joint_states_topic">/isaac_joint_states</param>
-                </xacro:if>
+              <plugin>gz_ros2_control/GazeboSimSystem</plugin>
             </hardware>
             <joint name="panda_joint1">

File: src/robot_arm/panda_description/urdf/panda.urdf.xacro (robot description, xacro)
@@ -5,4 +5,17 @@
 <!-- =================================================================================== -->
 <robot name="panda" xmlns:xacro="http://www.ros.org/wiki/xacro">
+  <xacro:arg name="robot_name" default="panda"/>
+  <xacro:arg name="use_gazebo" default="true"/>
+  <xacro:arg name="use_camera" default="false"/>
+  <xacro:arg name="add_world" default="true"/>
+  <!-- World link -->
+  <xacro:if value="$(arg add_world)">
+    <link name="world"/>
+    <joint name="world_to_panda_link0" type="fixed">
+      <parent link="world"/>
+      <child link="panda_link0"/>
+      <origin xyz="0 0 0" rpy="0 0 0"/>
+    </joint>
+  </xacro:if>
     <link name="panda_link0">
         <visual>
@@ -286,3 +299,13 @@
         <dynamics damping="0.3" />
     </joint>
-</robot>
+    <xacro:include filename="$(find panda_description)/urdf/control/gazebo_sim_ros2_control.urdf.xacro" />
+    <xacro:load_gazebo_sim_ros2_control_plugin
+    robot_name="$(arg robot_name)"
+    use_gazebo="$(arg use_gazebo)"/>
+    <xacro:include filename="$(find panda_description)/urdf/control/panda_ros2_control.urdf.xacro" />
+    <xacro:panda_ros2_control
+    name="PandaSystem"
+    initial_positions_file="$(find panda_moveit_config)/config/initial_positions.yaml"
+    ros2_control_hardware_type="gz_ros2_control/GazeboSimSystem"
+    use_gazebo="$(arg use_gazebo)"/>
+ </robot>
