Commit message: Stable Gazebo for BB01, Moveit Config and Multi Arduino Test
Implemented many things

File: src/robot_arm/robot_description/robots/bb01/urdf/bb01.urdf (robot description, URDF)
Before this commit: robot BB01_URDF, 8 links, 7 joints
Joints:
- joint joint_1: limit lower=0 upper=0 effort=0 velocity=0 -> lower=-1.5707963267948966 upper=1.5707963267948966 effort=10 velocity=10
- joint joint_2: limit lower=0 upper=0 effort=0 velocity=0 -> lower=-1.5707963267948966 upper=1.5707963267948966 effort=10 velocity=10
- joint joint_3: limit lower=0 upper=0 effort=0 velocity=0 -> lower=-1.5707963267948966 upper=1.5707963267948966 effort=10 velocity=10
- joint joint_4: limit lower=0 upper=0 effort=0 velocity=0 -> lower=-1.5707963267948966 upper=1.5707963267948966 effort=10 velocity=10
- joint joint_5: limit lower=0 upper=0 effort=0 velocity=0 -> lower=-1.5707963267948966 upper=1.5707963267948966 effort=10 velocity=10
- joint joint_6: limit lower=0 upper=0 effort=0 velocity=0 -> lower=-1.5707963267948966 upper=1.5707963267948966 effort=10 velocity=10

File: src/robot_arm/robot_description/robots/bb01/urdf/control/bb01_ros2_control.urdf.xacro (robot description, xacro)
@@ -2,5 +2,4 @@
 <robot xmlns:xacro="http://www.ros.org/wiki/xacro" name="bb01_description">
     <xacro:macro name="bb01_ros2_control" params="use_gazebo">
-    <xacro:property name="PI" value="3.1415926535897931"/>
         <ros2_control type="system" name="BB01System">
             <hardware>
@@ -11,49 +10,43 @@
             <joint name="joint_1">
                 <command_interface name="position">
-                    <param name="min">-${PI/2}</param>
-                    <param name="max">${PI/2}</param>
+                    <param name="min">-1.570795</param>
+                    <param name="max">1.570795</param>
                 </command_interface>
                 <state_interface name="position"/>
-                <state_interface name="velocity"/>
             </joint>
             <joint name="joint_2">
                 <command_interface name="position">
-                    <param name="min">-${PI/2}</param>
-                    <param name="max">${PI/2}</param>
+                    <param name="min">-1.570795</param>
+                    <param name="max">1.570795</param>
                 </command_interface>
                 <state_interface name="position"/>
-                <state_interface name="velocity"/>
             </joint>
             <joint name="joint_3">
                 <command_interface name="position">
-                    <param name="min">-${PI/2}</param>
-                    <param name="max">${PI/2}</param>
+                    <param name="min">-1.570795</param>
+                    <param name="max">1.570795</param>
                 </command_interface>
                 <state_interface name="position"/>
-                <state_interface name="velocity"/>
             </joint>
             <joint name="joint_4">
                 <command_interface name="position">
-                    <param name="min">-${PI/2}</param>
-                    <param name="max">${PI/2}</param>
+                    <param name="min">-1.570795</param>
+                    <param name="max">1.570795</param>
                 </command_interface>
                 <state_interface name="position"/>
-                <state_interface name="velocity"/>
             </joint>
             <joint name="joint_5">
                 <command_interface name="position">
-                    <param name="min">-${PI/2}</param>
-                    <param name="max">${PI/2}</param>
+                    <param name="min">-1.570795</param>
+                    <param name="max">1.570795</param>
                 </command_interface>
                 <state_interface name="position"/>
-                <state_interface name="velocity"/>
             </joint>
             <joint name="joint_6">
                 <command_interface name="position">
-                    <param name="min">-${PI/2}</param>
-                    <param name="max">${PI/2}</param>
+                    <param name="min">-1.570795</param>
+                    <param name="max">1.570795</param>
                 </command_interface>
                 <state_interface name="position"/>
-                <state_interface name="velocity"/>
             </joint>
         </ros2_control>

File: src/robot_arm/robot_description/robots/bb01/urdf/control/gazebo_sim_ros2_control.urdf.xacro (robot description, xacro)
@@ -5,5 +5,5 @@
             <gazebo>
                 <plugin filename="gz_ros2_control-system" name="gz_ros2_control::GazeboSimROS2ControlPlugin">
-                    <parameters>$(find robot_description)/robots/bb01/config/ros2_controllers.yaml</parameters>
+                    <parameters>$(find bb01_moveit_config)/config/ros2_controllers.yaml</parameters>
                     <ros>
                         <remapping>/controller_manager/robot_description:=/robot_description</remapping>

Commit message: Stable Moveit for BB01 - Work on meshes pending
working with cube collision meshes

File: src/robot_arm/robot_description/robots/bb01/urdf/bb01.urdf (robot description, URDF)
Before this commit: robot bb01, 8 links, 7 joints
Joints:
- removed joint world_to_base_link
- added joint virtual_joint: type fixed, parent world, child base_link, origin xyz=0 0 0 rpy=0 0 0

File: src/robot_arm/robot_description/robots/bb01/urdf/bb01.urdf.xacro (robot description, xacro)
@@ -3,4 +3,5 @@
      Commit Version: 1.6.0-4-g7f85cfe  Build Version: 1.6.7995.38578
      For more information, please see http://wiki.ros.org/sw_urdf_exporter -->
+  <!-- NOTE: Collision geometry uses simplified boxes instead of high-poly meshes to prevent MoveIt startup timeout/freeze. -->
 <robot name="bb01" xmlns:xacro="http://www.ros.org/wiki/xacro">
   <xacro:arg name="add_world" default="true"/>
@@ -13,6 +14,6 @@
   <xacro:if value="$(arg add_world)">
     <link name="world"/>
-    <!-- Fixed joint connecting world to base_link -->
-    <joint name="world_to_base_link" type="fixed">
+    <!-- Fixed joint connecting world to base_link (named virtual_joint to match SRDF) -->
+    <joint name="virtual_joint" type="fixed">
       <parent link="world"/>
       <child link="base_link"/>
@@ -55,6 +56,5 @@
         rpy="0 0 0" />
       <geometry>
-        <mesh
-          filename="package://robot_description/robots/bb01/meshes/base_link.STL" />
+        <box size="0.1 0.1 0.1"/>
       </geometry>
     </collision>
@@ -95,6 +95,5 @@
         rpy="0 0 0" />
       <geometry>
-        <mesh
-          filename="package://robot_description/robots/bb01/meshes/link_1.STL" />
+        <box size="0.1 0.1 0.1"/>
       </geometry>
     </collision>
@@ -115,5 +114,5 @@
       lower="${-PI/2}"
       upper="${PI/2}"
-      effort="10"
+      effort="46.74"
       velocity="10" />
   </joint>
@@ -153,6 +152,5 @@
         rpy="0 0 0" />
       <geometry>
-        <mesh
-          filename="package://robot_description/robots/bb01/meshes/link_2.STL" />
+        <box size="0.1 0.1 0.1"/>
       </geometry>
     </collision>
@@ -173,5 +171,5 @@
       lower="${-PI/2}"
       upper="${PI/2}"
-      effort="10"
+      effort="41.82"
       velocity="10" />
   </joint>
@@ -211,6 +209,5 @@
         rpy="0 0 0" />
       <geometry>
-        <mesh
-          filename="package://robot_description/robots/bb01/meshes/link_3.STL" />
+        <box size="0.1 0.1 0.1"/>
       </geometry>
     </collision>
@@ -231,5 +228,5 @@
       lower="${-PI/2}"
       upper="${PI/2}"
-      effort="10"
+      effort="24.27"
       velocity="10" />
   </joint>
@@ -269,6 +266,5 @@
         rpy="0 0 0" />
       <geometry>
-        <mesh
-          filename="package://robot_description/robots/bb01/meshes/link_4.STL" />
+        <box size="0.1 0.1 0.1"/>
       </geometry>
     </collision>
@@ -289,5 +285,5 @@
       lower="${-PI/2}"
       upper="${PI/2}"
-      effort="10"
+      effort="1.85"
       velocity="10" />
   </joint>
@@ -327,6 +323,5 @@
         rpy="0 0 0" />
       <geometry>
-        <mesh
-          filename="package://robot_description/robots/bb01/meshes/link_5.STL" />
+        <box size="0.1 0.1 0.1"/>
       </geometry>
     </collision>
@@ -347,5 +342,5 @@
       lower="${-PI/2}"
       upper="${PI/2}"
-      effort="10"
+      effort="2.03"
       velocity="10" />
   </joint>
@@ -385,6 +380,5 @@
         rpy="0 0 0" />
       <geometry>
-        <mesh
-          filename="package://robot_description/robots/bb01/meshes/link_6.STL" />
+        <box size="0.1 0.1 0.1"/>
       </geometry>
     </collision>
@@ -405,5 +399,5 @@
       lower="${-PI/2}"
       upper="${PI/2}"
-      effort="10"
+      effort="0.45"
       velocity="10" />
   </joint>
