Commit message: Implemented and validated all URDFs and launch files

File: src/robot_arm/robot_description/robots/bb01/urdf/bb01.urdf.xacro (robot description, xacro)
@@ -3,14 +3,21 @@
      Commit Version: 1.6.0-4-g7f85cfe  Build Version: 1.6.7995.38578
      For more information, please see http://wiki.ros.org/sw_urdf_exporter -->
-<robot
-  name="BB01_URDF">
+<robot name="bb01" xmlns:xacro="http://www.ros.org/wiki/xacro">
+  <xacro:arg name="add_world" default="true"/>
+  <xacro:arg name="robot_name" default="bb01"/>
+  <xacro:arg name="use_gazebo" default="true"/>
+  <xacro:arg name="use_camera" default="false"/>
+  <!-- Constants -->
+  <xacro:property name="PI" value="3.1415926535897931"/>
   <!-- World link (root link with no inertia to fix KDL parser warning) -->
-  <link name="world"/>
-  <!-- Fixed joint connecting world to base_link -->
-  <joint name="world_to_base_link" type="fixed">
-    <parent link="world"/>
-    <child link="base_link"/>
-    <origin xyz="0 0 0" rpy="0 0 0"/>
-  </joint>
+  <xacro:if value="$(arg add_world)">
+    <link name="world"/>
+    <!-- Fixed joint connecting world to base_link -->
+    <joint name="world_to_base_link" type="fixed">
+      <parent link="world"/>
+      <child link="base_link"/>
+      <origin xyz="0 0 0" rpy="0 0 0"/>
+    </joint>
+  </xacro:if>
   <link
     name="base_link">
@@ -106,6 +113,6 @@
       xyz="0.0010187 -0.0029659 1" />
     <limit
-      lower="0"
-      upper="0"
+      lower="${-PI/2}"
+      upper="${PI/2}"
       effort="0"
       velocity="0" />
@@ -164,6 +171,6 @@
       xyz="0.014776 -0.99989 -0.0029807" />
     <limit
-      lower="0"
-      upper="0"
+      lower="${-PI/2}"
+      upper="${PI/2}"
       effort="0"
       velocity="0" />
@@ -222,6 +229,6 @@
       xyz="-0.014776 0.99989 0.0029807" />
     <limit
-      lower="0"
-      upper="0"
+      lower="${-PI/2}"
+      upper="${PI/2}"
       effort="0"
       velocity="0" />
@@ -280,6 +287,6 @@
       xyz="0.014776 -0.99989 -0.0029807" />
     <limit
-      lower="0"
-      upper="0"
+      lower="${-PI/2}"
+      upper="${PI/2}"
       effort="0"
       velocity="0" />
@@ -338,6 +345,6 @@
       xyz="0.010953 -0.0028189 0.99994" />
     <limit
-      lower="0"
-      upper="0"
+      lower="${-PI/2}"
+      upper="${PI/2}"
       effort="0"
       velocity="0" />
@@ -396,6 +403,6 @@
       xyz="-0.014776 0.99989 0.0029807" />
     <limit
-      lower="0"
-      upper="0"
+      lower="${-PI/2}"
+      upper="${PI/2}"
       effort="0"
       velocity="0" />

Commit message: Fixed Gazebo Launch
Pending fix for controlers launch. Added intial ESP32 with microros code

File: src/robot_arm/robot_description/robots/bb01/urdf/bb01.urdf.xacro (robot description, xacro)
@@ -115,6 +115,6 @@
       lower="${-PI/2}"
       upper="${PI/2}"
-      effort="0"
-      velocity="0" />
+      effort="10"
+      velocity="10" />
   </joint>
   <link
@@ -173,6 +173,6 @@
       lower="${-PI/2}"
       upper="${PI/2}"
-      effort="0"
-      velocity="0" />
+      effort="10"
+      velocity="10" />
   </joint>
   <link
@@ -231,6 +231,6 @@
       lower="${-PI/2}"
       upper="${PI/2}"
-      effort="0"
-      velocity="0" />
+      effort="10"
+      velocity="10" />
   </joint>
   <link
@@ -289,6 +289,6 @@
       lower="${-PI/2}"
       upper="${PI/2}"
-      effort="0"
-      velocity="0" />
+      effort="10"
+      velocity="10" />
   </joint>
   <link
@@ -347,6 +347,6 @@
       lower="${-PI/2}"
       upper="${PI/2}"
-      effort="0"
-      velocity="0" />
+      effort="10"
+      velocity="10" />
   </joint>
   <link
@@ -405,6 +405,15 @@
       lower="${-PI/2}"
       upper="${PI/2}"
-      effort="0"
-      velocity="0" />
-  </joint>
+      effort="10"
+      velocity="10" />
+  </joint>
+  <!-- Include Gazebo ros2_control plugin -->
+  <xacro:include filename="$(find robot_description)/robots/bb01/urdf/control/gazebo_sim_ros2_control.urdf.xacro" />
+  <xacro:load_gazebo_sim_ros2_control_plugin
+      robot_name="$(arg robot_name)"
+      use_gazebo="$(arg use_gazebo)"/>
+  <!-- Include ros2_control joint interfaces -->
+  <xacro:include filename="$(find robot_description)/robots/bb01/urdf/control/bb01_ros2_control.urdf.xacro" />
+  <xacro:bb01_ros2_control
+      use_gazebo="$(arg use_gazebo)"/>
 </robot>

Commit message: Stable working moveit for bb01

File: src/robot_arm/robot_description/robots/bb01/urdf/bb01.urdf.xacro (robot description, xacro)
@@ -3,5 +3,5 @@
      Commit Version: 1.6.0-4-g7f85cfe  Build Version: 1.6.7995.38578
      For more information, please see http://wiki.ros.org/sw_urdf_exporter -->
-  <!-- NOTE: Collision geometry uses simplified boxes instead of high-poly meshes to prevent MoveIt startup timeout/freeze. -->
+  <!-- NOTE: Collision geometry uses dedicated collision meshes for accurate collision detection. -->
 <robot name="bb01" xmlns:xacro="http://www.ros.org/wiki/xacro">
   <xacro:arg name="add_world" default="true"/>
@@ -56,5 +56,6 @@
         rpy="0 0 0" />
       <geometry>
-        <box size="0.1 0.1 0.1"/>
+        <mesh
+          filename="package://robot_description/robots/bb01/meshes/collision_base_link.STL" />
       </geometry>
     </collision>
@@ -95,5 +96,6 @@
         rpy="0 0 0" />
       <geometry>
-        <box size="0.1 0.1 0.1"/>
+        <mesh
+          filename="package://robot_description/robots/bb01/meshes/collision_link_1.STL" />
       </geometry>
     </collision>
@@ -152,5 +154,6 @@
         rpy="0 0 0" />
       <geometry>
-        <box size="0.1 0.1 0.1"/>
+        <mesh
+          filename="package://robot_description/robots/bb01/meshes/collision_link_2.STL" />
       </geometry>
     </collision>
@@ -209,5 +212,6 @@
         rpy="0 0 0" />
       <geometry>
-        <box size="0.1 0.1 0.1"/>
+        <mesh
+          filename="package://robot_description/robots/bb01/meshes/collision_link_3.STL" />
       </geometry>
     </collision>
@@ -266,5 +270,6 @@
         rpy="0 0 0" />
       <geometry>
-        <box size="0.1 0.1 0.1"/>
+        <mesh
+          filename="package://robot_description/robots/bb01/meshes/collision_link_4.STL" />
       </geometry>
     </collision>
@@ -323,5 +328,6 @@
         rpy="0 0 0" />
       <geometry>
-        <box size="0.1 0.1 0.1"/>
+        <mesh
+          filename="package://robot_description/robots/bb01/meshes/collision_link_5.STL" />
       </geometry>
     </collision>
@@ -380,5 +386,6 @@
         rpy="0 0 0" />
       <geometry>
-        <box size="0.1 0.1 0.1"/>
+        <mesh
+          filename="package://robot_description/robots/bb01/meshes/collision_link_6.STL" />
       </geometry>
     </collision>
